Commit message: feat: Implement SLAM, Nav2, and Gazebo simulation bringup by adding launch/config files and updating dependencies.

File: src/robot_description/urdf/AEP_Robot_macro.urdf.xacro (robot description, xacro)
@@ -1,4 +1,6 @@
 <?xml version="1.0"?>
 <robot xmlns:xacro="http://www.ros.org/wiki/xacro">
+  <!-- Define mesh path - use file:// for Gazebo compatibility -->
+  <xacro:property name="mesh_path" value="file://$(find robot_description)/meshes"/>
   <xacro:macro name="AEP_Robot" params="prefix:=">
     <!-- base_link -->
@@ -18,5 +20,5 @@
         <origin xyz="0 0 0" rpy="0 0 0" />
         <geometry>
-          <mesh filename="package://robot_description/meshes/base_link.STL" />
+          <mesh filename="${mesh_path}/base_link.STL" />
         </geometry>
         <material name="">
@@ -27,5 +29,5 @@
         <origin xyz="0 0 0" rpy="0 0 0" />
         <geometry>
-          <mesh filename="package://robot_description/meshes/base_link.STL" />
+          <mesh filename="${mesh_path}/base_link.STL" />
         </geometry>
       </collision>
@@ -47,5 +49,5 @@
         <origin xyz="0 0 0" rpy="0 0 0" />
         <geometry>
-          <mesh filename="package://robot_description/meshes/lidar_link.STL" />
+          <mesh filename="${mesh_path}/lidar_link.STL" />
         </geometry>
         <material name="">
@@ -56,5 +58,5 @@
         <origin xyz="0 0 0" rpy="0 0 0" />
         <geometry>
-          <mesh filename="package://robot_description/meshes/lidar_link.STL" />
+          <mesh filename="${mesh_path}/lidar_link.STL" />
         </geometry>
       </collision>
@@ -82,5 +84,5 @@
         <origin xyz="0 0 0" rpy="0 0 0" />
         <geometry>
-          <mesh filename="package://robot_description/meshes/left_wheel_link.STL" />
+          <mesh filename="${mesh_path}/left_wheel_link.STL" />
         </geometry>
         <material name="">
@@ -91,5 +93,5 @@
         <origin xyz="0 0 0" rpy="0 0 0" />
         <geometry>
-          <mesh filename="package://robot_description/meshes/left_wheel_link.STL" />
+          <mesh filename="${mesh_path}/left_wheel_link.STL" />
         </geometry>
       </collision>
@@ -100,5 +102,5 @@
       <child  link="${prefix}left_wheel_link" />
       <axis xyz="0 1 0" />
-      <limit lower="0" upper="0" effort="0" velocity="0" />
+      <limit effort="20.0" velocity="10.0" />
     </joint>
     <!-- right wheel -->
@@ -118,5 +120,5 @@
         <origin xyz="0 0 0" rpy="0 0 0" />
         <geometry>
-          <mesh filename="package://robot_description/meshes/right_wheel_link.STL" />
+          <mesh filename="${mesh_path}/right_wheel_link.STL" />
         </geometry>
         <material name="">
@@ -127,5 +129,5 @@
         <origin xyz="0 0 0" rpy="0 0 0" />
         <geometry>
-          <mesh filename="package://robot_description/meshes/right_wheel_link.STL" />
+          <mesh filename="${mesh_path}/right_wheel_link.STL" />
         </geometry>
       </collision>
@@ -136,5 +138,5 @@
       <child  link="${prefix}right_wheel_link" />
       <axis xyz="0 1 0" />
-      <limit lower="0" upper="0" effort="0" velocity="0" />
+      <limit effort="20.0" velocity="10.0" />
     </joint>
     <!-- front caster -->
@@ -154,5 +156,5 @@
         <origin xyz="0 0 0" rpy="0 0 0" />
         <geometry>
-          <mesh filename="package://robot_description/meshes/front_castor_body_link.STL" />
+          <mesh filename="${mesh_path}/front_castor_body_link.STL" />
         </geometry>
         <material name="">
@@ -163,5 +165,5 @@
         <origin xyz="0 0 0" rpy="0 0 0" />
         <geometry>
-          <mesh filename="package://robot_description/meshes/front_castor_body_link.STL" />
+          <mesh filename="${mesh_path}/front_castor_body_link.STL" />
         </geometry>
       </collision>
@@ -189,5 +191,5 @@
         <origin xyz="0 0 0" rpy="0 0 0" />
         <geometry>
-          <mesh filename="package://robot_description/meshes/front_castor_wheel_link.STL" />
+          <mesh filename="${mesh_path}/front_castor_wheel_link.STL" />
         </geometry>
         <material name="">
@@ -198,5 +200,5 @@
         <origin xyz="0 0 0" rpy="0 0 0" />
         <geometry>
-          <mesh filename="package://robot_description/meshes/front_castor_wheel_link.STL" />
+          <mesh filename="${mesh_path}/front_castor_wheel_link.STL" />
         </geometry>
       </collision>
@@ -225,5 +227,5 @@
         <origin xyz="0 0 0" rpy="0 0 0" />
         <geometry>
-          <mesh filename="package://robot_description/meshes/back_castor_body_link.STL" />
+          <mesh filename="${mesh_path}/back_castor_body_link.STL" />
         </geometry>
         <material name="">
@@ -234,5 +236,5 @@
         <origin xyz="0 0 0" rpy="0 0 0" />
         <geometry>
-          <mesh filename="package://robot_description/meshes/back_castor_body_link.STL" />
+          <mesh filename="${mesh_path}/back_castor_body_link.STL" />
         </geometry>
       </collision>
@@ -260,5 +262,5 @@
         <origin xyz="0 0 0" rpy="0 0 0" />
         <geometry>
-          <mesh filename="package://robot_description/meshes/back_castor_wheel_link.STL" />
+          <mesh filename="${mesh_path}/back_castor_wheel_link.STL" />
         </geometry>
         <material name="">
@@ -269,5 +271,5 @@
         <origin xyz="0 0 0" rpy="0 0 0" />
         <geometry>
-          <mesh filename="package://robot_description/meshes/back_castor_wheel_link.STL" />
+          <mesh filename="${mesh_path}/back_castor_wheel_link.STL" />
         </geometry>
       </collision>
@@ -280,4 +282,70 @@
       <limit lower="0" upper="0" effort="0" velocity="0" />
     </joint>
+    <!-- ==================== GAZEBO PLUGINS ==================== -->
+    <!-- Differential Drive Plugin -->
+    <gazebo>
+      <plugin filename="gz-sim-diff-drive-system" name="gz::sim::systems::DiffDrive">
+        <left_joint>${prefix}left_wheel_joint</left_joint>
+        <right_joint>${prefix}right_wheel_joint</right_joint>
+        <wheel_separation>0.5897</wheel_separation>
+        <wheel_radius>0.10</wheel_radius>
+        <max_wheel_torque>20.0</max_wheel_torque>
+        <max_wheel_acceleration>1.0</max_wheel_acceleration>
+        <odom_publish_frequency>50</odom_publish_frequency>
+        <topic>cmd_vel</topic>
+        <odom_topic>odom</odom_topic>
+        <tf_topic>tf</tf_topic>
+        <frame_id>odom</frame_id>
+        <child_frame_id>${prefix}base_link</child_frame_id>
+      </plugin>
+    </gazebo>
+    <!-- Joint State Publisher Plugin -->
+    <gazebo>
+      <plugin filename="gz-sim-joint-state-publisher-system" name="gz::sim::systems::JointStatePublisher">
+        <joint_name>${prefix}left_wheel_joint</joint_name>
+        <joint_name>${prefix}right_wheel_joint</joint_name>
+        <joint_name>${prefix}front_castor_body_joint</joint_name>
+        <joint_name>${prefix}front_castor_wheel_joint</joint_name>
+        <joint_name>${prefix}back_castor_body_joint</joint_name>
+        <joint_name>${prefix}back_castor_wheel_joint</joint_name>
+        <topic>joint_states</topic>
+      </plugin>
+    </gazebo>
+    <!-- GPU Lidar Sensor -->
+    <gazebo reference="${prefix}lidar_link">
+      <sensor name="gpu_lidar" type="gpu_lidar">
+        <pose>0 0 0 0 0 0</pose>
+        <topic>scan</topic>
+        <update_rate>10</update_rate>
+        <lidar>
+          <scan>
+            <horizontal>
+              <samples>360</samples>
+              <resolution>1</resolution>
+              <min_angle>-3.14159</min_angle>
+              <max_angle>3.14159</max_angle>
+            </horizontal>
+            <vertical>
+              <samples>1</samples>
+              <resolution>1</resolution>
+              <min_angle>0</min_angle>
+              <max_angle>0</max_angle>
+            </vertical>
+          </scan>
+          <range>
+            <min>0.1</min>
+            <max>12.0</max>
+            <resolution>0.01</resolution>
+          </range>
+          <noise>
+            <type>gaussian</type>
+            <mean>0.0</mean>
+            <stddev>0.01</stddev>
+          </noise>
+        </lidar>
+        <always_on>true</always_on>
+        <visualize>true</visualize>
+      </sensor>
+    </gazebo>
   </xacro:macro>
 </robot>

Commit message: Add TurtleBot3 simulation and SLAM toolbox integration
- Created a new launch file for TurtleBot3 simulation (`turtlebot3_sim.launch.py`) that sets up the robot description, Gazebo simulation, and SLAM toolbox.
- Added a new URDF file for TurtleBot3 with Ignition Gazebo plugins (`turtlebot3_waffle_gz.urdf.xacro`).
- Introduced a complex world SDF file (`complex_world.sdf`) with various obstacles for testing.
- Implemented SLAM toolbox configuration files, including launch and parameter files for online asynchronous SLAM.
- Added scripts for converting odometry to pose, extracting ground truth from Ignition, and transforming TF to pose.
- Created a package for the SLAM toolbox with necessary dependencies and configurations.
- Updated topics list to include relevant topics for the simulation and SLAM processes.

File: src/robot_description/urdf/AEP_Robot_macro.urdf.xacro (robot description, xacro)
@@ -27,7 +27,7 @@
       </visual>
       <collision>
-        <origin xyz="0 0 0" rpy="0 0 0" />
-        <geometry>
-          <mesh filename="${mesh_path}/base_link.STL" />
+        <origin xyz="0 0 0.05" rpy="0 0 0" />
+        <geometry>
+          <box size="0.5 0.35 0.2" />
         </geometry>
       </collision>
@@ -91,10 +91,14 @@
       </visual>
       <collision>
-        <origin xyz="0 0 0" rpy="0 0 0" />
-        <geometry>
-          <mesh filename="${mesh_path}/left_wheel_link.STL" />
-        </geometry>
-      </collision>
-    </link>
+        <origin xyz="0 0 0" rpy="1.570796 0 0" />
+        <geometry>
+          <cylinder radius="0.075" length="0.04"/>
+        </geometry>
+      </collision>
+    </link>
+    <gazebo reference="${prefix}left_wheel_link">
+      <mu1>1.0</mu1>
+      <mu2>1.0</mu2>
+    </gazebo>
     <joint name="${prefix}left_wheel_joint" type="continuous">
       <origin xyz="0 0.29485 -0.025" rpy="0 0 0" />
@@ -127,10 +131,14 @@
       </visual>
       <collision>
-        <origin xyz="0 0 0" rpy="0 0 0" />
-        <geometry>
-          <mesh filename="${mesh_path}/right_wheel_link.STL" />
-        </geometry>
-      </collision>
-    </link>
+        <origin xyz="0 0 0" rpy="1.570796 0 0" />
+        <geometry>
+          <cylinder radius="0.075" length="0.04"/>
+        </geometry>
+      </collision>
+    </link>
+    <gazebo reference="${prefix}right_wheel_link">
+      <mu1>1.0</mu1>
+      <mu2>1.0</mu2>
+    </gazebo>
     <joint name="${prefix}right_wheel_joint" type="continuous">
       <origin xyz="0 -0.29485 -0.025" rpy="0 0 0" />
@@ -162,10 +170,11 @@
         </material>
       </visual>
-      <collision>
+      <!-- Collision removed to prevent ground dragging -->
+      <!-- <collision>
         <origin xyz="0 0 0" rpy="0 0 0" />
         <geometry>
           <mesh filename="${mesh_path}/front_castor_body_link.STL" />
         </geometry>
-      </collision>
+      </collision> -->
     </link>
     <joint name="${prefix}front_castor_body_joint" type="continuous">
@@ -200,8 +209,12 @@
         <origin xyz="0 0 0" rpy="0 0 0" />
         <geometry>
-          <mesh filename="${mesh_path}/front_castor_wheel_link.STL" />
-        </geometry>
-      </collision>
-    </link>
+          <sphere radius="0.0255"/>
+        </geometry>
+      </collision>
+    </link>
+    <gazebo reference="${prefix}front_castor_wheel_link">
+      <mu1>0.01</mu1>
+      <mu2>0.01</mu2>
+    </gazebo>
     <joint name="${prefix}front_castor_wheel_joint" type="continuous">
       <origin xyz="0.021643 0.023336 -0.033" rpy="0 0 0" />
@@ -233,10 +246,11 @@
         </material>
       </visual>
-      <collision>
+      <!-- Collision removed to prevent ground dragging -->
+      <!-- <collision>
         <origin xyz="0 0 0" rpy="0 0 0" />
         <geometry>
           <mesh filename="${mesh_path}/back_castor_body_link.STL" />
         </geometry>
-      </collision>
+      </collision> -->
     </link>
     <joint name="${prefix}back_castor_body_joint" type="continuous">
@@ -271,8 +285,12 @@
         <origin xyz="0 0 0" rpy="0 0 0" />
         <geometry>
-          <mesh filename="${mesh_path}/back_castor_wheel_link.STL" />
-        </geometry>
-      </collision>
-    </link>
+          <sphere radius="0.0255"/>
+        </geometry>
+      </collision>
+    </link>
+    <gazebo reference="${prefix}back_castor_wheel_link">
+      <mu1>0.01</mu1>
+      <mu2>0.01</mu2>
+    </gazebo>
     <joint name="${prefix}back_castor_wheel_joint" type="continuous">
       <origin xyz="-0.024216 0.020654 -0.033" rpy="0 0 0" />
