Commit message: refactor: Restructure robot simulation, description, bringup, SLAM, and navigation packages by deleting numerous old files, modifying existing URDFs and configs, and introducing new launch files and configurations for

File: src/robot_description/urdf/AEP_Robot_macro.urdf.xacro (robot description, xacro)
@@ -1,12 +1,312 @@
 <?xml version="1.0"?>
 <robot xmlns:xacro="http://www.ros.org/wiki/xacro">
+  <!-- Define mesh path - use file:// for Gazebo compatibility -->
+  <xacro:property name="mesh_path" value="file://$(find robot_description)/meshes"/>
   <xacro:macro name="AEP_Robot" params="prefix:=">
-    <!-- Gazebo joint state publisher (MODEL SCOPE) -->
+    <!-- base_link -->
+    <link name="${prefix}base_link">
+      <inertial>
+        <origin xyz="-0.0023189 0.0073427 0.1843" rpy="0 0 0" />
+        <mass value="15.896" />
+        <inertia
+          ixx="0.65725"
+          ixy="-3.6456E-08"
+          ixz="0.040641"
+          iyy="0.58335"
+          iyz="-2.2784E-12"
+          izz="0.1582" />
+      </inertial>
+      <visual>
+        <origin xyz="0 0 0" rpy="0 0 0" />
+        <geometry>
+          <mesh filename="${mesh_path}/base_link.STL" />
+        </geometry>
+        <material name="">
+          <color rgba="0.5 0.5 0.5 1" />
+        </material>
+      </visual>
+      <collision>
+        <origin xyz="0 0 0" rpy="0 0 0" />
+        <geometry>
+          <mesh filename="${mesh_path}/base_link.STL" />
+        </geometry>
+      </collision>
+    </link>
+    <!-- lidar -->
+    <link name="${prefix}lidar_link">
+      <inertial>
+        <origin xyz="-9.1926E-05 -0.0067665 -0.0073819" rpy="0 0 0" />
+        <mass value="1.3308" />
+        <inertia
+          ixx="0.0009607"
+          ixy="8.0198E-07"
+          ixz="-3.0916E-06"
+          iyy="0.00061492"
+          iyz="-0.00015824"
+          izz="0.0010982" />
+      </inertial>
+      <visual>
+        <origin xyz="0 0 0" rpy="0 0 0" />
+        <geometry>
+          <mesh filename="${mesh_path}/lidar_link.STL" />
+        </geometry>
+        <material name="">
+          <color rgba="0.2 0.7 1 1" />
+        </material>
+      </visual>
+      <collision>
+        <origin xyz="0 0 0" rpy="0 0 0" />
+        <geometry>
+          <mesh filename="${mesh_path}/lidar_link.STL" />
+        </geometry>
+      </collision>
+    </link>
+    <joint name="${prefix}lidar_joint" type="fixed">
+      <origin xyz="0 0.000420393431200835 0.32565" rpy="0 0 0" />
+      <parent link="${prefix}base_link" />
+      <child  link="${prefix}lidar_link" />
+      <axis xyz="0 0 0" />
+    </joint>
+    <!-- left wheel -->
+    <link name="${prefix}left_wheel_link">
+      <inertial>
+        <origin xyz="8.211E-08 -0.017522 -4.1793E-07" rpy="0 0 0" />
+        <mass value="0.583" />
+        <inertia
+          ixx="0.00092026"
+          ixy="2.1255E-10"
+          ixz="8.2654E-07"
+          iyy="0.0017198"
+          iyz="-1.099E-09"
+          izz="0.00091447" />
+      </inertial>
+      <visual>
+        <origin xyz="0 0 0" rpy="0 0 0" />
+        <geometry>
+          <mesh filename="${mesh_path}/left_wheel_link.STL" />
+        </geometry>
+        <material name="">
+          <color rgba="0.7 0.1 0.8 1" />
+        </material>
+      </visual>
+      <collision>
+        <origin xyz="0 0 0" rpy="0 0 0" />
+        <geometry>
+          <mesh filename="${mesh_path}/left_wheel_link.STL" />
+        </geometry>
+      </collision>
+    </link>
+    <joint name="${prefix}left_wheel_joint" type="continuous">
+      <origin xyz="0 0.29485 -0.025" rpy="0 0 0" />
+      <parent link="${prefix}base_link" />
+      <child  link="${prefix}left_wheel_link" />
+      <axis xyz="0 1 0" />
+      <limit effort="20.0" velocity="10.0" />
+    </joint>
+    <!-- right wheel -->
+    <link name="${prefix}right_wheel_link">
+      <inertial>
+        <origin xyz="3.8174E-07 0.017522 1.8833E-07" rpy="0 0 0" />
+        <mass value="0.583" />
+        <inertia
+          ixx="0.00091579"
+          ixy="-1.3235E-09"
+          ixz="-2.5693E-06"
+          iyy="0.0017198"
+          iyz="-7.3676E-10"
+          izz="0.00091893" />
+      </inertial>
+      <visual>
+        <origin xyz="0 0 0" rpy="0 0 0" />
+        <geometry>
+          <mesh filename="${mesh_path}/right_wheel_link.STL" />
+        </geometry>
+        <material name="">
+          <color rgba="0.7 0.1 0.8 1" />
+        </material>
+      </visual>
+      <collision>
+        <origin xyz="0 0 0" rpy="0 0 0" />
+        <geometry>
+          <mesh filename="${mesh_path}/right_wheel_link.STL" />
+        </geometry>
+      </collision>
+    </link>
+    <joint name="${prefix}right_wheel_joint" type="continuous">
+      <origin xyz="0 -0.29485 -0.025" rpy="0 0 0" />
+      <parent link="${prefix}base_link" />
+      <child  link="${prefix}right_wheel_link" />
+      <axis xyz="0 1 0" />
+      <limit effort="20.0" velocity="10.0" />
+    </joint>
+    <!-- front caster -->
+    <link name="${prefix}front_castor_body_link">
+      <inertial>
+        <origin xyz="0.0055133 0.00033058 -0.0066169" rpy="0 0 0" />
+        <mass value="0.011291" />
+        <inertia
+          ixx="4.0603E-06"
+          ixy="1.367E-08"
+          ixz="8.6782E-07"
+          iyy="3.8335E-06"
+          iyz="5.2075E-08"
+          izz="4.4634E-06" />
+      </inertial>
+      <visual>
+        <origin xyz="0 0 0" rpy="0 0 0" />
+        <geometry>
+          <mesh filename="${mesh_path}/front_castor_body_link.STL" />
+        </geometry>
+        <material name="">
+          <color rgba="0.4 0.4 0.4 1" />
+        </material>
+      </visual>
+      <collision>
+        <origin xyz="0 0 0" rpy="0 0 0" />
+        <geometry>
+          <mesh filename="${mesh_path}/front_castor_body_link.STL" />
+        </geometry>
+      </collision>
+    </link>
+    <joint name="${prefix}front_castor_body_joint" type="continuous">
+      <origin xyz="0.105 0 -0.0415" rpy="0 0 0" />
+      <parent link="${prefix}base_link" />
+      <child  link="${prefix}front_castor_body_link" />
+      <axis xyz="0 0 1" />
+      <limit lower="0" upper="0" effort="0" velocity="0" />
+    </joint>
+    <link name="${prefix}front_castor_wheel_link">
+      <inertial>
+        <origin xyz="0.001327 -0.02196 3.518E-06" rpy="0 0 0" />
+        <mass value="0.047259" />
+        <inertia
+          ixx="9.5221E-06"
+          ixy="-2.7895E-07"
+          ixz="2.5434E-09"
+          iyy="1.4162E-05"
+          iyz="1.5234E-10"
+          izz="9.4977E-06" />
+      </inertial>
+      <visual>
+        <origin xyz="0 0 0" rpy="0 0 0" />
+        <geometry>
+          <mesh filename="${mesh_path}/front_castor_wheel_link.STL" />
+        </geometry>
+        <material name="">
+          <color rgba="0.6 0.6 0.6 1" />
+        </material>
+      </visual>
+      <collision>
+        <origin xyz="0 0 0" rpy="0 0 0" />
+        <geometry>
+          <mesh filename="${mesh_path}/front_castor_wheel_link.STL" />
+        </geometry>
+      </collision>
+    </link>
+    <joint name="${prefix}front_castor_wheel_joint" type="continuous">
+      <origin xyz="0.021643 0.023336 -0.033" rpy="0 0 0" />
+      <parent link="${prefix}front_castor_body_link" />
+      <child  link="${prefix}front_castor_wheel_link" />
+      <axis xyz="0 1 0" />
+      <limit lower="0" upper="0" effort="0" velocity="0" />
+    </joint>
+    <!-- back caster -->
+    <link name="${prefix}back_castor_body_link">
+      <inertial>
+        <origin xyz="-0.0055142 -0.00031498 -0.0066169" rpy="0 0 0" />
+        <mass value="0.011291" />
+        <inertia
+          ixx="4.0603E-06"
+          ixy="1.3028E-08"
+          ixz="-8.6797E-07"
+          iyy="3.8334E-06"
+          iyz="-4.9618E-08"
+          izz="4.4634E-06" />
+      </inertial>
+      <visual>
+        <origin xyz="0 0 0" rpy="0 0 0" />
+        <geometry>
+          <mesh filename="${mesh_path}/back_castor_body_link.STL" />
+        </geometry>
+        <material name="">
+          <color rgba="0.4 0.4 0.4 1" />
+        </material>
+      </visual>
+      <collision>
+        <origin xyz="0 0 0" rpy="0 0 0" />
+        <geometry>
+          <mesh filename="${mesh_path}/back_castor_body_link.STL" />
+        </geometry>
+      </collision>
+    </link>
+    <joint name="${prefix}back_castor_body_joint" type="continuous">
+      <origin xyz="-0.105 0 -0.0415" rpy="0 0 0" />
+      <parent link="${prefix}base_link" />
+      <child  link="${prefix}back_castor_body_link" />
+      <axis xyz="0 0 1" />
+      <limit lower="0" upper="0" effort="0" velocity="0" />
+    </joint>
+    <link name="${prefix}back_castor_wheel_link">
+      <inertial>
+        <origin xyz="0.001265 -0.021964 -2.6984E-06" rpy="0 0 0" />
+        <mass value="0.047259" />
+        <inertia
+          ixx="9.5208E-06"
+          ixy="-2.6579E-07"
+          ixz="-1.9877E-09"
+          iyy="1.4164E-05"
+          iyz="-1.1341E-10"
+          izz="9.4974E-06" />
+      </inertial>
+      <visual>
+        <origin xyz="0 0 0" rpy="0 0 0" />
+        <geometry>
+          <mesh filename="${mesh_path}/back_castor_wheel_link.STL" />
+        </geometry>
+        <material name="">
+          <color rgba="0.6 0.6 0.6 1" />
+        </material>
+      </visual>
+      <collision>
+        <origin xyz="0 0 0" rpy="0 0 0" />
+        <geometry>
+          <mesh filename="${mesh_path}/back_castor_wheel_link.STL" />
+        </geometry>
+      </collision>
+    </link>
+    <joint name="${prefix}back_castor_wheel_joint" type="continuous">
+      <origin xyz="-0.024216 0.020654 -0.033" rpy="0 0 0" />
+      <parent link="${prefix}back_castor_body_link" />
+      <child  link="${prefix}back_castor_wheel_link" />
+      <axis xyz="0 1 0" />
+      <limit lower="0" upper="0" effort="0" velocity="0" />
+    </joint>
+    <!-- ==================== GAZEBO PLUGINS ==================== -->
+    <!-- Differential Drive Plugin -->
     <gazebo>
-      <plugin filename="ignition-gazebo-joint-state-publisher-system"
-          name="ignition::gazebo::systems::JointStatePublisher">
-        <!-- Use a clear gazebo topic name -->
-        <topic>/joint_states</topic>
-        <!-- Publish only the joints you want -->
+      <plugin filename="gz-sim-diff-drive-system" name="gz::sim::systems::DiffDrive">
+        <left_joint>${prefix}left_wheel_joint</left_joint>
+        <right_joint>${prefix}right_wheel_joint</right_joint>
+        <wheel_separation>0.5897</wheel_separation>
+        <wheel_radius>0.075</wheel_radius>
+        <max_wheel_torque>20.0</max_wheel_torque>
+        <max_wheel_acceleration>1.0</max_wheel_acceleration>
+        <odom_publish_frequency>50</odom_publish_frequency>
+        <topic>cmd_vel</topic>
+        <odom_topic>odom</odom_topic>
+        <tf_topic>tf</tf_topic>
+        <frame_id>odom</frame_id>
+        <child_frame_id>${prefix}base_link</child_frame_id>
+      </plugin>
+    </gazebo>
+    <!-- Sensors System Plugin (required for GPU lidar) -->
+    <gazebo>
+      <plugin filename="gz-sim-sensors-system" name="gz::sim::systems::Sensors">
+        <render_engine>ogre2</render_engine>
+      </plugin>
+    </gazebo>
+    <!-- Joint State Publisher Plugin -->
+    <gazebo>
+      <plugin filename="gz-sim-joint-state-publisher-system" name="gz::sim::systems::JointStatePublisher">
         <joint_name>${prefix}left_wheel_joint</joint_name>
         <joint_name>${prefix}right_wheel_joint</joint_name>
@@ -15,309 +315,44 @@
         <joint_name>${prefix}back_castor_body_joint</joint_name>
         <joint_name>${prefix}back_castor_wheel_joint</joint_name>
+        <topic>joint_states</topic>
       </plugin>
     </gazebo>
-    <!-- base_footprint (root, no inertial) -->
-    <link name="${prefix}base_footprint" />
-    <!-- base_link -->
-    <link name="${prefix}base_link">
-      <inertial>
-        <origin xyz="-0.0023189 0.0073427 0.1843" rpy="0 0 0" />
-        <mass value="15.896" />
-        <inertia ixx="0.65725" ixy="-3.6456E-08" ixz="0.040641" iyy="0.58335" iyz="-2.2784E-12" izz="0.1582" />
-      </inertial>
-      <visual>
-        <origin xyz="0 0 0" rpy="0 0 0" />
-        <geometry>
-          <mesh filename="package://robot_description/meshes/base_link.STL" />
-        </geometry>
-        <material name="">
-          <color rgba="0.5 0.5 0.5 1" />
-        </material>
-      </visual>
-      <collision>
-        <origin xyz="0 0 0" rpy="0 0 0" />
-        <geometry>
-          <mesh filename="package://robot_description/meshes/base_link.STL" />
-        </geometry>
-      </collision>
-    </link>
-    <joint name="${prefix}base_footprint_joint" type="fixed">
-      <origin xyz="0 0 0" rpy="0 0 0" />
-      <parent link="${prefix}base_footprint" />
-      <child link="${prefix}base_link" />
-    </joint>
-    <!-- Gazebo diff-drive plugin (MODEL SCOPE) -->
-    <gazebo>
-      <plugin name="ignition::gazebo::systems::DiffDrive" filename="ignition-gazebo-diff-drive-system">
-        <left_joint>${prefix}left_wheel_joint</left_joint>
-        <right_joint>${prefix}right_wheel_joint</right_joint>
-        <wheel_separation>0.5897</wheel_separation>
-        <wheel_radius>0.1</wheel_radius>
-        <odom_publish_frequency>50</odom_publish_frequency>
-        <!-- cmd vel in Gazebo -->
-        <topic>/cmd_vel</topic>
-        <!-- Odometry output in Gazebo (TF disabled; use ROS TF only) -->
-        <odom_topic>/odom</odom_topic>
-      </plugin>
+    <!-- GPU Lidar Sensor -->
+    <gazebo reference="${prefix}lidar_link">
+      <sensor name="gpu_lidar" type="gpu_lidar">
+        <pose>0 0 0 0 0 0</pose>
+        <topic>scan</topic>
+        <update_rate>10</update_rate>
+        <gz_frame_id>${prefix}lidar_link</gz_frame_id>
+        <lidar>
+          <scan>
+            <horizontal>
+              <samples>360</samples>
+              <resolution>1</resolution>
+              <min_angle>-3.14159</min_angle>
+              <max_angle>3.14159</max_angle>
+            </horizontal>
+            <vertical>
+              <samples>1</samples>
+              <resolution>1</resolution>
+              <min_angle>0</min_angle>
+              <max_angle>0</max_angle>
+            </vertical>
+          </scan>
+          <range>
+            <min>0.1</min>
+            <max>12.0</max>
+            <resolution>0.01</resolution>
+          </range>
+          <noise>
+            <type>gaussian</type>
+            <mean>0.0</mean>
+            <stddev>0.01</stddev>
+          </noise>
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
File: src/robot_description/urdf/main.urdf.xacro (robot description, xacro)
@@ -1,5 +1,5 @@
 <?xml version="1.0"?>
 <robot name="AEP_Robot" xmlns:xacro="http://www.ros.org/wiki/xacro">
-  <xacro:include filename="AEP_Robot_macro.urdf.xacro"/>
+  <xacro:include filename="$(find robot_description)/urdf/AEP_Robot_macro.urdf.xacro"/>
   <xacro:AEP_Robot prefix=""/>
 </robot>
